Commit message: h1 added, tocabi(bug remain)

File: resources/robots/bolt6/urdf/bolt6.urdf (robot description, URDF)
Before this commit: robot bolt, 9 links, 8 joints
Joints:
- joint FL_HFE: limit lower=-1.57 upper=1.57 effort=2.5 velocity=20 -> lower=-1.57 upper=0.0 effort=2.5 velocity=20
- joint FR_HFE: limit lower=-1.57 upper=1.57 effort=2.5 velocity=20 -> lower=-1.57 upper=0.0 effort=2.5 velocity=20
